File: hardware/kicad/tellmelight_rev_a2/tellmelight_rev_a2.kicad_pcb (KiCad board)
At the start: 4 copper layers, 96 x 74 mm, 56 parts, among them J1 USB_C, SW1 BOOT, SW2 RESET, U1 RP2040, U2 LP5024, U3 W25Q32JVSS, U4 AP2112K-3.3, U5 TPD2EUSB30, Y1 12MHz

Commit message: feat: map rev a2 rgb led footprint
Parts:
- D1, D2, D3, D4, D5, D6: footprint LED_RGB_Wuerth-PLCC4_3.2x2.8mm_150141M173100 -> LED_RGB_TUOZHAN_S4-3528RGBTA-A_3.5x2.8mm
Other:
- board text added: "Check JLC LED orientation"
- board text removed: "Do not order: LED pinout RED"
