File: hardware/kicad/tellmelight_rev_a2/tellmelight_rev_a2.kicad_sch (KiCad schematic)
At the start: 20 parts, among them J1 USB_C_Receptacle_USB2.0, SW1 BOOT, SW2 RESET, U1 RP2040, U2 LP5024RSMR, U3 W25Q32JVSSIQ, U4 AP2112K-3.3TRG1, U5 TPD2EUSB30DRTR, Y1 12MHz

Commit message: feat: map rev a2 rgb led footprint
Parts:
- D1, D2, D3, D4, D5, D6: footprint LED_SMD:LED_RGB_Wuerth-PLCC4_3.2x2.8mm_150141M173100 -> TellMeLight_Rev_A2:LED_RGB_TUOZHAN_S4-3528RGBTA-A_3.5x2.8mm
Changed lines of the file:
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@@
 			)
 		)
-		(property "Footprint" "LED_SMD:LED_RGB_Wuerth-PLCC4_3.2x2.8mm_150141M173100"
+		(property "Footprint" "TellMeLight_Rev_A2:LED_RGB_TUOZHAN_S4-3528RGBTA-A_3.5x2.8mm"
 			(at 105 178 0)
 			(effects
@@
 			)
 		)
-		(property "Footprint" "LED_SMD:LED_RGB_Wuerth-PLCC4_3.2x2.8mm_150141M173100"
+		(property "Footprint" "TellMeLight_Rev_A2:LED_RGB_TUOZHAN_S4-3528RGBTA-A_3.5x2.8mm"
 			(at 145 178 0)
 			(effects
@@
 			)
 		)
-		(property "Footprint" "LED_SMD:LED_RGB_Wuerth-PLCC4_3.2x2.8mm_150141M173100"
+		(property "Footprint" "TellMeLight_Rev_A2:LED_RGB_TUOZHAN_S4-3528RGBTA-A_3.5x2.8mm"
 			(at 25 198 0)
 			(effects
@@
 			)
 		)
-		(property "Footprint" "LED_SMD:LED_RGB_Wuerth-PLCC4_3.2x2.8mm_150141M173100"
+		(property "Footprint" "TellMeLight_Rev_A2:LED_RGB_TUOZHAN_S4-3528RGBTA-A_3.5x2.8mm"
 			(at 65 198 0)
 			(effects
@@
 			)
 		)
-		(property "Footprint" "LED_SMD:LED_RGB_Wuerth-PLCC4_3.2x2.8mm_150141M173100"
+		(property "Footprint" "TellMeLight_Rev_A2:LED_RGB_TUOZHAN_S4-3528RGBTA-A_3.5x2.8mm"
 			(at 105 198 0)
 			(effects
@@
 			)
 		)
-		(property "Footprint" "LED_SMD:LED_RGB_Wuerth-PLCC4_3.2x2.8mm_150141M173100"
+		(property "Footprint" "TellMeLight_Rev_A2:LED_RGB_TUOZHAN_S4-3528RGBTA-A_3.5x2.8mm"
 			(at 145 198 0)
 			(effects
