File: hardware/kicad/tellmelight_rev_a4/tellmelight_rev_a4.kicad_pcb (KiCad board)
At the start: 4 copper layers, 76 x 56 mm, 61 parts, among them J1 USB_C, SW1 BOOT, SW2 RESET, U1 RP2040, U2 LP5024, U3 W25Q32JVSS, U4 AP2112K-3.3, U5 TPD2EUSB30, U6 TPD1E05U06DPY, Y1 12MHz

Commit message: hardware: finish rev a4 routing preview package
Parts:
- moved C7 14.0 mm to (42.0, 44.5)
- moved R1 13.0 mm to (45.0, 44.0)
- moved R2 13.0 mm to (49.0, 44.0)
- moved R10 6.00 mm to (53.0, 45.0)
- moved R7 5.66 mm to (30.0, 32.0)
- moved C15 5.00 mm to (35.0, 31.0)
- moved C18 1.58 mm to (46.5, 40.5)
Routing:
- net RUN_RESET: track 24.5 -> 100.8 mm, vias 0 -> 3
- net 3V3: track 134.7 -> 184.5 mm, vias 0 -> 9
- net SWDIO: track 0.00 -> 42.3 mm, vias 0 -> 2
- net SWCLK: track 0.00 -> 37.6 mm, vias 0 -> 2
- net GND: track 240.3 -> 275.4 mm, vias 0 -> 7
- net LP_EN: track 0.00 -> 22.3 mm, vias 0 -> 3
- net FLASH_WP_IO2: track 0.00 -> 21.9 mm, vias 0 -> 2
- net FLASH_IO0_MOSI: track 0.00 -> 20.9 mm, vias 0 -> 2
- net FLASH_IO1_MISO: track 0.00 -> 19.8 mm, vias 0 -> 2
- net XIN: track 4.26 -> 24.0 mm, vias 0 -> 2
- net FLASH_HOLD_IO3: track 0.00 -> 19.4 mm, vias 0 -> 2
- net FLASH_SCLK: track 0.00 -> 19.4 mm, vias 0 -> 2
- net D3_R: track 0.00 -> 18.4 mm, vias 0 -> 1
- net I2C0_SDA: track 47.5 -> 65.7 mm, vias 2 -> 3
- net USB_DM_CONN: track 50.7 -> 65.6 mm, vias 3 -> 4
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- removed copper zone on B.Cu, net 3V3
- removed copper zone on B.Cu, net GND
- removed copper zone on In2.Cu, net GND

Commit message: hardware: correct rev a4 ordinary via routing
Routing:
- net GND: track 275.4 -> 248.4 mm, vias 7 -> 4
- net USB_DP_CONN: track 54.0 -> 63.0 mm, vias 2 -> 0
- net VLED: track 138.3 -> 132.5 mm, vias 5 -> 6
- net VBUS: track 98.5 -> 103.6 mm, vias 3 -> 4
- net USB_DM_CONN: track 65.6 -> 70.2 mm, vias 4 -> 2
- net SWCLK: track 37.6 -> 42.1 mm
- net FLASH_IO0_MOSI: track 20.9 -> 16.8 mm, vias 2 -> 1
- net D3_R: track 18.4 -> 14.3 mm, vias 1 -> 2
- net I2C0_SCL: track 70.1 -> 66.3 mm, vias 4 -> 3
- net D2_B: track 35.6 -> 32.5 mm, vias 1 -> 2
- net D1_R: track 35.4 -> 32.7 mm, vias 2 -> 1
- net D4_G: track 14.8 -> 12.3 mm
- net RP2040_VREG_OUT: track 11.4 -> 9.18 mm, vias 2 -> 1
- net LP_EN: track 22.3 -> 20.3 mm
- net XIN: track 24.0 -> 22.1 mm
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
Commit message: hardware: align rev a4 with JLC free vias
Parts:
- U1: footprint QFN-56-1EP_7x7mm_P0.4mm_EP3.2x3.2mm_ThermalVias -> QFN-56-1EP_7x7mm_P0.4mm_EP3.2x3.2mm
- U2: footprint VQFN-32-1EP_4x4mm_P0.4mm_EP2.8x2.8mm_ThermalVias -> VQFN-32-1EP_4x4mm_P0.4mm_EP2.8x2.8mm
Routing:
- net VLED: track 132.5 -> 143.9 mm, vias 6 -> 5
- net 3V3: track 186.2 -> 194.5 mm, vias 12 -> 11
- net FLASH_IO1_MISO: track 20.9 -> 28.5 mm
- net USB_DM_CONN: track 70.2 -> 64.6 mm, vias 2 -> 3
- net SWCLK: track 42.1 -> 36.7 mm
- net RUN_RESET: track 99.0 -> 93.7 mm, vias 3 -> 5
- net GND: track 248.4 -> 253.0 mm
- net D3_B: track 23.3 -> 20.0 mm
- net D1_G: track 34.6 -> 31.6 mm
- net D4_B: track 19.4 -> 16.5 mm, vias 1 -> 2
- net FLASH_CS_N_BOOTSEL: track 49.5 -> 52.4 mm, vias 4 -> 3
- net SHIELD: track 48.9 -> 46.6 mm
- net USB_DP_CONN: track 63.0 -> 60.8 mm, vias 0 -> 2
- net USB_DP_MCU: track 10.1 -> 12.2 mm
- net D1_B: track 30.3 -> 32.4 mm, vias 1 -> 2
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